File: Schematic/LED_Panel_v3/LED_Panel_v3.sch (KiCad schematic (older format))
At the start: 9 parts

Commit message: saving everything on local repo
Parts:
- added C1: 10uF, symbol Device:C
- added C2, C? (x7): 0.1uF, symbol Device:C
- added C3, C5, C6, C7, C8, C9, C? (x2): 47uF, symbol Device:C
- added D1: Royal Blue, symbol Device:LED
- added D11: Deep Blue, symbol Device:LED
- added D13, D14: Violet, symbol Device:LED
- added D15, D16, D17: Cyan, symbol Device:LED
- added D18, D19, D20: UV, symbol Device:LED
- added D21, D22, D23: Red, symbol Device:LED
- added D24, D25, D26, D27: Green, symbol Device:LED
- added Q1, Q3, Q4, Q5, Q6, Q7, Q? (x2): IRLB8721PBF, Package_TO_SOT_THT:TO-220-3_Vertical, symbol Transistor_FET:IRLB8721PBF
- added R1, R4, R5, R6, R7, R8, R? (x2): 1, symbol Device:R_US
- added R2: 5.1K, symbol Device:R_US
- added RV1, RV? (x7): 500k 20T, symbol Device:R_POT_US
- added U1, U2, U3, U? (x3): MCP6004, symbol Amplifier_Operational:MCP6004
- gave numbers to parts that had none: 9
Connections:
- net VCC: now reaches D2.2 (A)
- net VCC: now also D24.2 (A)
- net at D10.1 (K): now also C3.1, Q1.2 (D)
- new net: Q1.1 (G), U1.1
- new net: Q1.3 (S), R1.1, U1.2 (-)
- new net: C2.1, RV1.2, U1.3 (+)
- new net: C1.1, R2.1, U?.3 (+)
- new net: C?.1, RV?.2, U2.5 (+)
- new net: Q3.3 (S), R4.1, U2.6 (-)
- new net: Q3.1 (G), U2.7
- new net: D24.1 (K), D25.2 (A)
- new net: D25.1 (K), D26.2 (A)
- new net: D26.1 (K), D27.2 (A)
- new net: C?.1, D27.1 (K), Q?.2 (D)
- new net: D21.1 (K), D22.2 (A)
- new net: D22.1 (K), D23.2 (A)
- new net: C9.1, D23.1 (K), Q7.2 (D)
- new net: D18.1 (K), D19.2 (A)
- new net: D19.1 (K), D20.2 (A)
- new net: C8.1, D20.1 (K), Q6.2 (D)
- new net: D15.1 (K), D16.2 (A)
- new net: D16.1 (K), D17.2 (A)
- new net: C6.1, D17.1 (K), Q4.2 (D)
- new net: D13.1 (K), D14.2 (A)
- new net: C5.1, D14.1 (K), Q3.2 (D)
- new net: C?.1, D11.1 (K), Q?.2 (D)
- new net: C7.1, D1.1 (K), Q5.2 (D)
- new net: Q5.1 (G), U2.1
- new net: Q5.3 (S), R6.1, U2.2 (-)
- new net: C?.1, RV?.2, U2.3 (+)
- new net: C?.1, RV?.2, U3.5 (+)
- new net: Q4.3 (S), R5.1, U3.6 (-)
- new net: Q4.1 (G), U3.7
- new net: C?.1, RV?.2, U3.10 (+)
- new net: Q6.1 (G), U3.8
- new net: Q6.3 (S), R7.1, U3.9 (-)
- new net: C?.1, RV?.2, U3.12 (+)
- new net: Q7.3 (S), R8.1, U3.13 (-)
- new net: Q7.1 (G), U3.14
- new net: Q?.1 (G), U?.1 (x2)
- new net: Q?.3 (S), R?.1, U?.2 (-) (x2)
- new net: C?.1, RV?.2, U?.3 (+) (x2)
- new net +10V: D15.2 (A), D21.2 (A)
- new net +12V: D18.2 (A)
- new net +5V: D1.2 (A), D11.2 (A)
- new net +9V: D13.2 (A)
- new net Driver: RV1.1, RV?.1, RV?.1, RV?.1, RV?.1, RV?.1, RV?.1, RV?.1, U?.1, U?.2 (-)
- new net GND: C1.2, C2.2, C3.2, C5.2, C6.2, C7.2, C8.2, C9.2, C?.2, C?.2, C?.2, C?.2, C?.2, C?.2, C?.2, C?.2, C?.2, R1.2, R4.2, R5.2, R6.2, R7.2, R8.2, R?.2, R?.2, RV1.3, RV?.3, RV?.3, RV?.3, RV?.3, RV?.3, RV?.3, RV?.3
- new net PWM: R2.2
Other:
- note added: "14V"
- note added: "26V"
- note added: "3"
- note added: "Solar Source Simulator Unit Panel"
- note added: "Solar Source Simulator \nUnit Panel"
- moved on the sheet: D10, D2, D3, D4, D5, D6, D7, D8, D9

Commit message: update fully
Parts:
- removed U? (x2): MCP6004, symbol Amplifier_Operational:MCP6004
- added C3: 0.1uF, symbol Device:C
- added C6: 47uF, symbol Device:C
- added LA1: Lamp, symbol Device:Lamp
- added Q2: IRLB8721PBF, Package_TO_SOT_THT:TO-220-3_Vertical, symbol Transistor_FET:IRLB8721PBF
- added R3: 1, symbol Device:R_US
- added RV2: 500k 20T, symbol Device:R_POT_US
- added unit 4 of U1
- added unit 2 of U1
- added unit 3 of U2
- gave numbers to parts that had none: 21
- renumbered C7 to C10, C8 to C12, C9 to C16, C2 to C17, C5 to C18, C3 to C19, C1 to C2, C6 to C8, D24 to D1, D19 to D10, D20 to D11, D11 to D12, D21 to D13, D22 to D14, D23 to D15, D13 to D16, D14 to D17, D2 to D18, D3 to D19, D25 to D2, D4 to D20, D5 to D21, D6 to D22, D7 to D23, D8 to D24, D9 to D25, D10 to D26, D26 to D3, D27 to D4, D15 to D5, D16 to D6, D17 to D7, D1 to D8, D18 to D9, Q4 to Q3, Q5 to Q4, Q6 to Q5, Q3 to Q8, Q1 to Q9, R2 to R1, R1 to R10, R5 to R4, R6 to R5, R7 to R6, R4 to R9, RV1 to RV9, U3 to U1, U1 to U2, U3 to U2, U2 to U3
Connections:
- net Driver: now also RV2.1
- net GND: now also C3.2, C6.2, R3.2, RV2.3
- net VCC: now also LA1.2 (+)
- net at U2.1: now also Q3.1 (G); no longer Q9.1 (G)
- net at Q9.3 (S), R10.1: now also U2.13 (-); no longer U2.2 (-)
- net at C17.1, RV9.2: now also U2.12 (+); no longer U2.3 (+)
- net at C15.1, RV8.2: now also U2.10 (+); no longer U3.5 (+)
- net at Q8.3 (S), R9.1: now also U2.9 (-); no longer U3.6 (-)
- net at U3.7: now also Q6.1 (G); no longer Q8.1 (G)
- net at C5.1, RV3.2: now also U2.3 (+); no longer U2.5 (+)
- net at Q3.3 (S), R4.1: now also U2.2 (-); no longer U2.6 (-)
- net at U2.7: now also Q5.1 (G); no longer Q3.1 (G)
- net at C9.1, RV5.2: now also U2.5 (+); no longer U1.10 (+)
- net at U1.8: now also Q7.1 (G); no longer Q5.1 (G)
- net at Q5.3 (S), R6.1: now also U2.6 (-); no longer U1.9 (-)
- net at C13.1, RV7.2: now also U1.10 (+); no longer U2.12 (+)
- net at Q7.3 (S), R8.1: now also U1.9 (-); no longer U2.13 (-)
- net at U2.14: now also Q9.1 (G); no longer Q7.1 (G)
- net at Q6.3 (S), R7.1: now also U3.6 (-)
- net at C11.1, RV6.2: now also U3.5 (+)
- net at Q1.1 (G): now also U1.14
- net at Q1.3 (S), R2.1: now also U1.13 (-)
- net at C1.1, RV1.2: now also U1.12 (+)
- new net: Q8.1 (G), U2.8
- new net: C6.1, LA1.1 (-), Q2.2 (D)
- new net: Q2.3 (S), R3.1, U1.6 (-)
- new net: Q2.1 (G), U1.7
- new net: C3.1, RV2.2, U1.5 (+)
Other:
- note added: "24V"
- note added: "4"
- note added: "6/10/20"
- note removed: "3"
- moved on the sheet: U1C, U2A, U2B, U2D, U3B
